Commit message: Updated Bunler description and add Pro description

File: bunker_description/urdf/bunker.urdf.xacro (robot description, xacro)
@@ -7,9 +7,4 @@
       </geometry>
     </visual>
-    <collision>
-      <geometry>
-        <mesh filename="package://bunker_description/meshes/Bunker_Tracks.dae"/>
-      </geometry>
-    </collision>
   </link>
   <joint name="base_link_joint" type="fixed">
@@ -24,9 +19,4 @@
       </geometry>
     </visual>
-    <collision>
-      <geometry>
-        <mesh filename="package://bunker_description/meshes/Bunker_Body.dae"/>
-      </geometry>
-    </collision>
   </link>
   <joint name="mid_mount_joint" type="fixed">
@@ -43,5 +33,5 @@
     <collision>
       <geometry>
-        <mesh filename="package://bunker_description/meshes/Bunker_Cover.dae"/>
+        <mesh filename="package://bunker_description/meshes/Bunker_Collision.stl"/>
       </geometry>
     </collision>

File: bunker_description/urdf/bunkerPro.urdf.xacro (robot description, xacro)
@@ -21,5 +21,5 @@
     <collision>
       <geometry>
-        <mesh filename="package://bunker_description/meshes/Bunker_Collision.dae"/>
+        <mesh filename="package://bunker_description/meshes/BunkerPro_Collision.stl"/>
       </geometry>
     </collision>
